File: sensorNode.sch (KiCad schematic (older format))
At the start: 20 parts, among them P1 PIR, P2 PRGM, P3 Serial I/O, SW1 Reset, U1 ESP-12, U2 DS18B20, U3 ISL29035

Commit message: Add part details for BOM
On branch newPCB
modified:   sensorNode.kicad_pcb
modified:   sensorNode.net
modified:   sensorNode.sch
modified:   sensorNode.xml
Parts:
- BT1: Characteristics (none) -> 2-AA; Description (none) -> HOLDER 2 CELL AA W/PC PINS; MFG (none) -> MPD (Memory Protection Devices); MFG P# (none) -> BA2AAPC; Notes (none) -> -; PN (none) -> BA2AAPC-ND; Pkg (none) -> -; Supplier (none) -> Digikey
- C1, C2: Characteristics (none) -> +/-10%, 16V; Description (none) -> CAP CER 0.1UF 16V 10% X7R 0603; MFG (none) -> Murata Electronics; MFG P# (none) -> GRM188R71C104KA01D; Notes (none) -> -; PN (none) -> 490-1532-1-ND; Pkg (none) -> 0603 (1608 Metric); Supplier (none) -> Digikey
- NT1, NT2: Characteristics (none) -> -; Description (none) -> -; MFG (none) -> -; MFG P# (none) -> -; Notes (none) -> -; PN (none) -> -; Pkg (none) -> -; Supplier (none) -> Digikey
- R1: Characteristics (none) -> +/-1%, 1/10W; Description (none) -> RES SMD 100 OHM 1% 1/10W 0603; MFG (none) -> Rohm; MFG P# (none) -> MCR03ERTF1000; Notes (none) -> -; PN (none) -> RHM100CFCT-ND; Pkg (none) -> 0603 (1608 Metric); Supplier (none) -> Digikey
- R2, R3: Characteristics (none) -> +/-1%, 1/10W; Description (none) -> RES SMD 10K OHM 1% 1/10W 0603; MFG (none) -> Rohm; MFG P# (none) -> MCR03EZPFX1002; Notes (none) -> -; PN (none) -> RHM10.0KHCT-ND; Pkg (none) -> 0603 (1608 Metric); Supplier (none) -> Digikey
- R4: Characteristics (none) -> +/-1%, 1/10W; Description (none) -> RES SMD 1K OHM 1% 1/10W 0603; MFG (none) -> Rohm; MFG P# (none) -> MCR03EZPFX1001; Notes (none) -> -; PN (none) -> RHM1.00KHCT-ND; Pkg (none) -> 0603 (1608 Metric); Supplier (none) -> Digikey
- R5, R6, R7, R8: Characteristics (none) -> +/-1%, 1/10W; Description (none) -> RES SMD 4.7K OHM 1% 1/10W 0603; MFG (none) -> Rohm Semiconductor; MFG P# (none) -> MCR03ERTF4701; Notes (none) -> -; PN (none) -> RHM4.70KCFCT-ND; Pkg (none) -> 0603 (1608 Metric); Supplier (none) -> Digikey
- SW1: Characteristics (none) -> Off-Mom; Description (none) -> SWITCH TACTILE SPST-NO 0.05A 12V; MFG (none) -> E-Switch; MFG P# (none) -> TL3302BF180QG/TR; Notes (none) -> -; PN (none) -> EG2529CT-ND; Pkg (none) -> http://spec_sheets.e-switch.com/specs/P010523.pdf; Supplier (none) -> Digikey
- U2: Characteristics (none) -> Sensor, Temperature; Description (none) -> SENSOR TEMPERATURE 1-WIRE TO92-3; MFG (none) -> Maxim Integrated; MFG P# (none) -> DS18B20+PAR; Notes (none) -> -; PN (none) -> DS18B20+PAR-ND; Pkg (none) -> TO-92-3; Supplier (none) -> Digikey
- U3: Characteristics (none) -> Sensor, Ambiant Light; Description (none) -> IC PROXIMITY SENSOR AMB LT 6ODFN; MFG (none) -> Intersil; MFG P# (none) -> ISL29035IROZ-T7; Notes (none) -> -; PN (none) -> ISL29035IROZ-T7CT-ND; Pkg (none) -> 6-ODFN (1.5x1.6); Supplier (none) -> Digikey
